File: kicad/3bp v2.1.kicad_pcb (KiCad board)
At the start: 2 copper layers, 29 x 38.5 mm, 86 parts, among them CON1 MD-90SM, U2 THS7374IPWR, U3 DMP-8

Commit message: added my modifications
Parts:
- removed the 1 at (-871.5, -657.5)
- removed the 1 at (-884.7, -657.6)
- removed the G at (-871.5, -654.7)
- removed the G at (-885.8, -680.6)
- removed JP1: JUMPER_SOLDER_1X2, easyeda:JUMPER_SOLDER_1X2
- removed the R1 at (-859.2, -651.7)
- removed the R1 at (-867.6, -662.0)
- removed U3: DMP-8, easyeda:DMP-8
- added 1: 3, easyeda:JUMPER, F.Cu at (140.6, 107.5)
- added 1: 3, easyeda:JUMPER, F.Cu at (127.4, 107.5)
- added ?: , , F.Cu at (151.9, 84.9)
- added ?: , , F.Cu at (142.9, 83.5)
- added ?: , , F.Cu at (145.0, 92.4)
- added ?: , , F.Cu at (151.9, 86.8)
- added ?: , , F.Cu at (127.0, 93.5)
- added ?: , , F.Cu at (125.3, 93.5)
- added ?: , , F.Cu at (151.9, 83.0)
- added ?: , , F.Cu at (127.0, 92.6)
- added ?: , , F.Cu at (145.0, 91.6)
- added ?: , , F.Cu at (125.3, 92.6)
- added C23: 47uF/10V, Capacitor_Tantalum_SMD:CP_EIA-3528-15_AVX-H, F.Cu at (127.4, 86.3)
- added G: LOGO, easyeda:OSHW-LOGO_5MM, F.Cu at (140.6, 110.4)
- added R1: 2.20k, Resistor_SMD:R_0603_1608Metric, F.Cu at (144.6, 105.8)
- added R38: 511, Resistor_SMD:R_0603_1608Metric, F.Cu at (149.3, 86.7)
- added R39: 511, Resistor_SMD:R_0603_1608Metric, F.Cu at (149.3, 84.9)
- added R40: 511, Resistor_SMD:R_0603_1608Metric, F.Cu at (149.3, 83.0)
- added R41: 1k, Resistor_SMD:R_0603_1608Metric, F.Cu at (126.1, 91.3)
- added R42: 1k, Resistor_SMD:R_0603_1608Metric, F.Cu at (126.1, 89.8)
- added RIN: TP_50, easyeda:TP50, F.Cu at (152.9, 113.4)
- added U1: TL972IDR, easyeda:DMP-8, F.Cu at (134.0, 99.2)
- C1, C10, C11, C12, C13, C14, C15, C20, C6: footprint easyeda:0603 -> Capacitor_SMD:C_0603_1608Metric
- C16, C9: value 0805 -> 10uF/16V; footprint easyeda:0805 -> Capacitor_SMD:C_0805_2012Metric
- C17: value 22uF/10V -> 10uF/16V; footprint easyeda:1206_P -> Capacitor_SMD:C_1206_3216Metric
- C18, C19: value 270pF/50V -> 150pF/50V; footprint easyeda:0603 -> Capacitor_SMD:C_0603_1608Metric
- C2, C3, C4, C5: value 270pF/50V -> 0.1uF/50V; footprint easyeda:0603 -> Capacitor_SMD:C_0603_1608Metric
- C21, C22: value CP_TANTALUM_CASE-B_EIA-3528-21_REFLOW -> 47uF/10V; footprint easyeda:CP_TANTALUM_CASE-B_EIA-3528-21_REFLOW -> Capacitor_Tantalum_SMD:CP_EIA-3528-15_AVX-H
- C7: footprint easyeda:1206_P -> Capacitor_SMD:C_1206_3216Metric
- C8: value CP_TANTALUM_CASE-B_EIA-3528-21_REFLOW -> 220uF/6.3V; footprint easyeda:CP_TANTALUM_CASE-B_EIA-3528-21_REFLOW -> Capacitor_Tantalum_SMD:CP_EIA-3528-15_AVX-H
- R10: value 1.00k -> 4.7k; footprint easyeda:0603 -> Resistor_SMD:R_0603_1608Metric
- R11: value 1.00k -> 75.0; footprint easyeda:0603 -> Resistor_SMD:R_0603_1608Metric
- R12, R13, R14, R17, R18, R19, R2, R3, R4, R5: footprint easyeda:0603 -> Resistor_SMD:R_0603_1608Metric
- R15: value 75.0 -> 2.20k; footprint easyeda:0603 -> Resistor_SMD:R_0603_1608Metric
- R16: value 75.0 -> 750; footprint easyeda:0603 -> Resistor_SMD:R_0603_1608Metric
- R20, R21, R24, R25: value 130k -> 210k; footprint easyeda:0603 -> Resistor_SMD:R_0603_1608Metric
- R22, R23: value 100k -> 210k; footprint easyeda:0603 -> Resistor_SMD:R_0603_1608Metric
- R26, R27: value 10.0k -> 10k; footprint easyeda:0603 -> Resistor_SMD:R_0603_1608Metric
- R28, R31: value 6.19k -> 130k; footprint easyeda:0603 -> Resistor_SMD:R_0603_1608Metric
- R29: value 130k -> 100k; footprint easyeda:0603 -> Resistor_SMD:R_0603_1608Metric
- R30: value 130k -> 10k; footprint easyeda:0603 -> Resistor_SMD:R_0603_1608Metric
- R32: value 6.19k -> 100k; footprint easyeda:0603 -> Resistor_SMD:R_0603_1608Metric
- R33: value 6.19k -> 10k; footprint easyeda:0603 -> Resistor_SMD:R_0603_1608Metric
- R34, R35: value 162k -> 300k; footprint easyeda:0603 -> Resistor_SMD:R_0603_1608Metric
- R36, R37: value 332 -> 330; footprint easyeda:0603 -> Resistor_SMD:R_0603_1608Metric
- R6, R7, R8, R9: value 1.00k -> 1k; footprint easyeda:0603 -> Resistor_SMD:R_0603_1608Metric
- moved R21 1270.8 mm to (141.8, 110.1), turned to 90 degrees
- moved C1 1270.8 mm to (144.2, 99.9), turned to 90 degrees
- moved C22 1270.7 mm to (130.9, 91.4)
- moved R28 1270.5 mm to (142.7, 103.4), turned to 90 degrees
- moved R26 1270.3 mm to (133.8, 104.3), turned to 90 degrees
- moved R37 1270.3 mm to (128.1, 95.4), turned to 180 degrees
- moved R8 1270.3 mm to (150.1, 102.9), turned to 90 degrees
- moved R11 1270.2 mm to (145.9, 90.3), turned to 0 degrees
- moved R22 1270.2 mm to (139.5, 110.1), turned to 90 degrees
- moved C20 1270.0 mm to (138.4, 95.4), turned to 180 degrees
- moved R24 1270.0 mm to (130.3, 110.1), turned to 90 degrees
- moved R9 1269.8 mm to (152.1, 102.9), turned to 90 degrees
- moved R34 1269.7 mm to (128.5, 98.3), turned to 90 degrees
- moved C11 1269.7 mm to (139.9, 113.9), turned to 90 degrees
- moved C15 1269.7 mm to (128.0, 114.0), turned to 90 degrees
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Connections:
- C8 pad 1: SYNC-OUT -> SYNC-75
- CON1 pad 6: NET-(CON101-PAD6) -> SM
- R11 pad 1: SYNC-OUT -> SYNC-75
Routing:
- net LEFT: track 34.4 -> 51.1 mm
- net SYNC-75: track 3.90 -> 18.2 mm, vias 0 -> 2
- net SM: track 0.00 -> 11.7 mm
- net B-OUT: track 13.3 -> 21.9 mm, vias 0 -> 2
- net GND: track 7.21 -> 0.44 mm, vias 26 -> 40
- net RIGHT: track 32.6 -> 38.2 mm
- net G-OUT: track 8.45 -> 13.1 mm
- net +5V: track 99.4 -> 95.0 mm
- net SYNC-OUT: track 63.8 -> 59.9 mm
- net R-OUT: track 8.09 -> 11.2 mm
- net LPF: track 5.94 -> 8.60 mm, vias 0 -> 2
Other:
- net class Default removed
- board text added: "2"
- board text added: "3BP V2-M by manadream"
- board text added: "BO"
- board text added: "Board remixed by manadream"
- board text added: "CVBS"
- board text added: "GO"
- board text added: "M1va0-6.5 = 1 M1va7 = 2 M2va0-1.8 = 2, c, e M2va2-2.3= 1, d-left M2va3 = 2 M2va4 = 3, d-right M3va1/2= 3, b, c, d-right, e, f"
- board text added: "RO"
- board text added: "S75"
- board text added: "SM"
- board text added: "SML"
- board text added: "SMR"
- board text added: "V2 board design by tianfeng33"
- board text removed: "Board design by"
- board text removed: "GND"
- board text removed: "LPF"
- board text removed: "M1va0-6.5= 1 M1va7 & M2va0-1.8= 2, c, d-right, e M2Va3= 2 M2va2-2.3= 1, d-left M2va4= 3, d-right M3va1/2= 3, b, c, d-right, e, f"
